File: keychain_game.kicad_pcb (KiCad board)
At the start: 2 copper layers, 28 parts, among them J1 Conn_02x03_Counter_Clockwise, J2 Conn_01x02, SW1 SW_MEC_5G, U1 MIC5205-2.5, U2 SN74HC595DR, U4 ATTINY13A-MMF

Commit message: updated schematic
Parts:
- moved R6 33.7 mm to (146.5, 102.5), turned to 270 degrees
- moved R9 33.4 mm to (139.4, 86.8), turned to 180 degrees
- moved D6 29.1 mm to (137.4, 92.3)
- moved R10 24.9 mm to (145.7, 81.3)
- moved D1 24.7 mm to (157.0, 84.2), turned to 45 degrees
- moved R3 24.4 mm to (151.6, 81.3)
- moved D5 24.3 mm to (140.2, 100.1), turned to 45 degrees
- moved C2 22.5 mm to (153.2, 102.0), turned to 25 degrees
- moved D3 20.6 mm to (157.7, 99.9), turned to 135 degrees
- moved R8 20.3 mm to (138.3, 89.8), turned to 180 degrees
- moved C4 19.6 mm to (141.1, 96.8), turned to 90 degrees
- moved R7 19.5 mm to (142.8, 101.6), turned to 180 degrees
- moved R1 17.5 mm to (140.5, 93.5), turned to 90 degrees
- moved D4 17.0 mm to (148.8, 103.8), turned to 90 degrees
- moved J1 15.2 mm to (157.3, 92.6)
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Routing:
- net Net-(D4-Pad2): track 0.00 -> 28.0 mm
- net +2V5: track 0.00 -> 21.8 mm
- net Net-(D3-Pad2): track 0.00 -> 21.7 mm
- net Net-(D5-Pad2): track 0.00 -> 20.9 mm
- net Net-(D2-Pad2): track 0.00 -> 13.6 mm
- net Net-(D6-Pad2): track 0.00 -> 13.1 mm
- net VCC: track 0.00 -> 10.2 mm, vias 0 -> 1
- net Net-(D7-Pad2): track 0.00 -> 5.89 mm
- net Net-(D8-Pad2): track 0.00 -> 4.94 mm
- net Net-(D3-Pad1): track 0.00 -> 4.90 mm
- net Net-(D7-Pad1): track 0.00 -> 4.12 mm
- net RESET: track 0.00 -> 3.96 mm
- net Net-(D6-Pad1): track 0.00 -> 2.85 mm
- net Net-(D4-Pad1): track 0.00 -> 2.82 mm
- net Net-(D5-Pad1): track 0.00 -> 2.59 mm
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Other:
- board outline added: 26.8 x 26.8 mm

Commit message: finished board
Parts:
- removed SW1: SW_MEC_5G, Button_Switch_SMD:SW_SPST_B3U-1000P
- added SW2: SW_DPST_x2, Button_Switch_SMD:SW_SPST_B3U-1000P, F.Cu at (149.1, 99.0)
- moved R5 1.13 mm to (160.0, 96.5)
- moved C1 0.78 mm to (155.2, 96.8)
- moved U4 0.49 mm to (148.7, 95.1)
- moved D8 0.40 mm to (149.1, 81.0)
- moved D5 0.23 mm to (140.4, 100.1)
- moved R4 0.09 mm to (160.4, 89.9), turned to 270 degrees
Connections:
- J1 pad 3: RCLK -> SCK
- U2 pad 11: MISO -> SCK
- U2 pad 12: RCLK -> MISO
- U4 pad 9: RCLK -> SCK
Routing:
- net GND: track 0.00 -> 33.5 mm, vias 0 -> 16
- net +2V5: track 21.8 -> 46.0 mm, vias 0 -> 2
- net RESET: track 3.96 -> 26.0 mm, vias 0 -> 2
- net SCK: track 0.00 -> 19.2 mm, vias 0 -> 2
- net Net-(R1-Pad1): track 0.00 -> 15.5 mm
- net Net-(D1-Pad2): track 0.00 -> 15.5 mm, vias 0 -> 2
- net MISO: track 0.00 -> 15.4 mm, vias 0 -> 2
- net VCC: track 10.2 -> 22.3 mm, vias 1 -> 2
- net MOSI: track 0.00 -> 10.5 mm, vias 0 -> 2
- net Net-(D1-Pad1): track 0.00 -> 5.26 mm
- net RCLK: track 2.51 -> 0.00 mm
- net Net-(D2-Pad1): track 0.00 -> 2.16 mm
- net Net-(D4-Pad2): track 28.0 -> 27.1 mm, vias 0 -> 2
- added copper zone on B.Cu, net GND
Other:
- board size 26.8 x 26.8 mm -> 26.4 x 26.4 mm
