File: keychain_game.kicad_pcb (KiCad board)
At the start: 2 copper layers, 26.4 x 26.4 mm, 28 parts, among them J1 Conn_02x03_Counter_Clockwise, J2 Conn_01x02, SW2 SW_DPST_x2, U1 MIC5205-2.5, U2 SN74HC595DR, U4 ATTINY13A-MMF

Commit message: updated desgin slightly
Parts:
- moved R5 0.41 mm to (159.6, 96.5)
Routing:
- net Net-(D3-Pad1): track 4.90 -> 3.36 mm
- net SCK: track 19.2 -> 18.1 mm
- net MISO: track 15.4 -> 15.5 mm, vias 2 -> 1
- net GND: vias 16 -> 15
- net VCC: vias 2 -> 1
