File: keychain_game.sch (KiCad schematic (older format))
At the start: 28 parts, among them J1 Conn_02x03_Counter_Clockwise, J2 Conn_01x02, SW1 SW_MEC_5G, U1 MIC5205-2.5, U2 SN74HC595DR, U3 ATTINY13A-MU

Commit message: updated schematic
Parts:
- C1, C2: footprint (none) -> Capacitors_Tantalum_SMD:CP_Tantalum_Case-B_EIA-3528-21_Reflow
- C3, C4: footprint (none) -> Capacitor_SMD:C_0603_1608Metric
- D1, D2, D3, D4, D5, D6, D7, D8: footprint (none) -> LED_SMD:LED_0603_1608Metric
- J1: footprint (none) -> Pin_Headers:Pin_Header_Straight_2x03_Pitch2.54mm; symbol Connector_Generic:Conn_02x03_Counter_Clockwise -> Connector_Generic:Conn_02x03_Odd_Even
- R1: footprint Battery_Holders:Keystone_3034_1x20mm-CoinCell -> Resistor_SMD:R_0805_2012Metric
- R10, R2, R3, R4, R5, R6, R7, R8, R9: footprint (none) -> Resistor_SMD:R_0805_2012Metric
- SW1: footprint (none) -> Buttons_Switches_SMD:SW_MEC_5GSH9
Connections:
- net GND: now also J1.6 (Pin_6); no longer J1.4 (Pin_4)
- net MOSI: now also J1.4 (Pin_4); no longer J1.5 (Pin_5)
- net RCLK: now also J1.3 (Pin_3); no longer J1.2 (Pin_2)
- net RESET: now also J1.5 (Pin_5); no longer J1.3 (Pin_3)
- net VCC: now also J1.2 (Pin_2); no longer J1.6 (Pin_6)
Changed lines of the file:
@@
 EESchema Schematic File Version 4
+LIBS:keychain_game-cache
 EELAYER 26 0
 EELAYER END
@@
 F 0 "D1" V 5095 1678 50  0000 L CNN
 F 1 "LED" V 5186 1678 50  0000 L CNN
-F 2 "" H 5150 1600 50  0001 C CNN
+F 2 "LED_SMD:LED_0603_1608Metric" H 5150 1600 50  0001 C CNN
 F 3 "~" H 5150 1600 50  0001 C CNN
 	1    5150 1600
@@
 F 0 "D2" V 5395 1678 50  0000 L CNN
 F 1 "LED" V 5486 1678 50  0000 L CNN
-F 2 "" H 5450 1600 50  0001 C CNN
+F 2 "LED_SMD:LED_0603_1608Metric" H 5450 1600 50  0001 C CNN
 F 3 "~" H 5450 1600 50  0001 C CNN
 	1    5450 1600
@@
 F 0 "D3" V 5695 1678 50  0000 L CNN
 F 1 "LED" V 5786 1678 50  0000 L CNN
-F 2 "" H 5750 1600 50  0001 C CNN
+F 2 "LED_SMD:LED_0603_1608Metric" H 5750 1600 50  0001 C CNN
 F 3 "~" H 5750 1600 50  0001 C CNN
 	1    5750 1600
@@
 F 0 "D4" V 5995 1678 50  0000 L CNN
 F 1 "LED" V 6086 1678 50  0000 L CNN
-F 2 "" H 6050 1600 50  0001 C CNN
+F 2 "LED_SMD:LED_0603_1608Metric" H 6050 1600 50  0001 C CNN
 F 3 "~" H 6050 1600 50  0001 C CNN
 	1    6050 1600
@@
 F 0 "D5" V 6295 1678 50  0000 L CNN
 F 1 "LED" V 6386 1678 50  0000 L CNN
-F 2 "" H 6350 1600 50  0001 C CNN
+F 2 "LED_SMD:LED_0603_1608Metric" H 6350 1600 50  0001 C CNN
 F 3 "~" H 6350 1600 50  0001 C CNN
 	1    6350 1600
@@
 F 0 "D6" V 6595 1678 50  0000 L CNN
 F 1 "LED" V 6686 1678 50  0000 L CNN
-F 2 "" H 6650 1600 50  0001 C CNN
+F 2 "LED_SMD:LED_0603_1608Metric" H 6650 1600 50  0001 C CNN
 F 3 "~" H 6650 1600 50  0001 C CNN
 	1    6650 1600
@@
 F 0 "D7" V 6895 1678 50  0000 L CNN
 F 1 "LED" V 6986 1678 50  0000 L CNN
-F 2 "" H 6950 1600 50  0001 C CNN
+F 2 "LED_SMD:LED_0603_1608Metric" H 6950 1600 50  0001 C CNN
 F 3 "~" H 6950 1600 50  0001 C CNN
 	1    6950 1600
@@
 F 0 "D8" V 7195 1678 50  0000 L CNN
 F 1 "LED" V 7286 1678 50  0000 L CNN
-F 2 "" H 7250 1600 50  0001 C CNN
+F 2 "LED_SMD:LED_0603_1608Metric" H 7250 1600 50  0001 C CNN
 F 3 "~" H 7250 1600 50  0001 C CNN
 	1    7250 1600
@@
 F 0 "R3" H 5220 1346 50  0000 L CNN
 F 1 "125" H 5220 1255 50  0000 L CNN
-F 2 "" V 5080 1300 50  0001 C CNN
+F 2 "Resistor_SMD:R_0805_2012Metric" V 5080 1300 50  0001 C CNN
 F 3 "~" H 5150 1300 50  0001 C CNN
 	1    5150 1300
@@
 F 0 "R4" H 5520 1346 50  0000 L CNN
 F 1 "125" H 5520 1255 50  0000 L CNN
-F 2 "" V 5380 1300 50  0001 C CNN
+F 2 "Resistor_SMD:R_0805_2012Metric" V 5380 1300 50  0001 C CNN
 F 3 "~" H 5450 1300 50  0001 C CNN
 	1    5450 1300
@@
 F 0 "R5" H 5820 1346 50  0000 L CNN
 F 1 "125" H 5820 1255 50  0000 L CNN
-F 2 "" V 5680 1300 50  0001 C CNN
+F 2 "Resistor_SMD:R_0805_2012Metric" V 5680 1300 50  0001 C CNN
 F 3 "~" H 5750 1300 50  0001 C CNN
 	1    5750 1300
@@
 F 0 "R6" H 6120 1346 50  0000 L CNN
 F 1 "125" H 6120 1255 50  0000 L CNN
-F 2 "" V 5980 1300 50  0001 C CNN
+F 2 "Resistor_SMD:R_0805_2012Metric" V 5980 1300 50  0001 C CNN
 F 3 "~" H 6050 1300 50  0001 C CNN
 	1    6050 1300
@@
 F 0 "R7" H 6420 1346 50  0000 L CNN
 F 1 "125" H 6420 1255 50  0000 L CNN
-F 2 "" V 6280 1300 50  0001 C CNN
+F 2 "Resistor_SMD:R_0805_2012Metric" V 6280 1300 50  0001 C CNN
 F 3 "~" H 6350 1300 50  0001 C CNN
 	1    6350 1300
@@
 F 0 "R8" H 6720 1346 50  0000 L CNN
 F 1 "125" H 6720 1255 50  0000 L CNN
-F 2 "" V 6580 1300 50  0001 C CNN
+F 2 "Resistor_SMD:R_0805_2012Metric" V 6580 1300 50  0001 C CNN
 F 3 "~" H 6650 1300 50  0001 C CNN
 	1    6650 1300
@@
 F 0 "R9" H 7020 1346 50  0000 L CNN
 F 1 "125" H 7020 1255 50  0000 L CNN
-F 2 "" V 6880 1300 50  0001 C CNN
+F 2 "Resistor_SMD:R_0805_2012Metric" V 6880 1300 50  0001 C CNN
 F 3 "~" H 6950 1300 50  0001 C CNN
 	1    6950 1300
@@
 F 0 "R10" H 7320 1346 50  0000 L CNN
 F 1 "125" H 7320 1255 50  0000 L CNN
-F 2 "" V 7180 1300 50  0001 C CNN
+F 2 "Resistor_SMD:R_0805_2012Metric" V 7180 1300 50  0001 C CNN
 F 3 "~" H 7250 1300 50  0001 C CNN
 	1    7250 1300
@@
 SER
 $Comp
-L Connector_Generic:Conn_02x03_Counter_Clockwise J1
+L Connector_Generic:Conn_02x03_Odd_Even J1
 U 1 1 5B7E6D36
 P 4000 5100
 F 0 "J1" H 4050 5417 50  0000 C CNN
 F 1 "Conn_02x03_Counter_Clockwise" H 4050 5326 50  0000 C CNN
-F 2 "" H 4000 5100 50  0001 C CNN
+F 2 "Pin_Headers:Pin_Header_Straight_2x03_Pitch2.54mm" H 4000 5100 50  0001 C CNN
 F 3 "~" H 4000 5100 50  0001 C CNN
 	1    4000 5100
@@
 F 0 "R1" V 1543 4550 50  0000 C CNN
 F 1 "10k" V 1634 4550 50  0000 C CNN
-F 2 "Battery_Holders:Keystone_3034_1x20mm-CoinCell" V 1680 4550 50  0001 C CNN
+F 2 "Resistor_SMD:R_0805_2012Metric" V 1680 4550 50  0001 C CNN
 F 3 "~" H 1750 4550 50  0001 C CNN
 	1    1750 4550
@@
 F 0 "SW1" V 2046 4702 50  0000 R CNN
 F 1 "SW_MEC_5G" V 1955 4702 50  0000 R CNN
-F 2 "" H 2000 4950 50  0001 C CNN
+F 2 "Buttons_Switches_SMD:SW_MEC_5GSH9" H 2000 4950 50  0001 C CNN
 F 3 "http://www.apem.com/int/index.php?controller=attachment&id_attachment=488" H 2000 4950 50  0001 C CNN
 	1    2000 4750
@@
 F 0 "R2" V 2493 4650 50  0000 C CNN
 F 1 "10k" V 2584 4650 50  0000 C CNN
-F 2 "" V 2630 4650 50  0001 C CNN
+F 2 "Resistor_SMD:R_0805_2012Metric" V 2630 4650 50  0001 C CNN
 F 3 "~" H 2700 4650 50  0001 C CNN
 	1    2700 4650
@@
 F 0 "C3" H 2842 1296 50  0000 L CNN
 F 1 ".1uF" H 2842 1205 50  0000 L CNN
-F 2 "" H 2750 1250 50  0001 C CNN
+F 2 "Capacitor_SMD:C_0603_1608Metric" H 2750 1250 50  0001 C CNN
 F 3 "~" H 2750 1250 50  0001 C CNN
 	1    2750 1250
@@
 F 0 "C4" H 5742 5046 50  0000 L CNN
 F 1 "0.1uF" H 5742 4955 50  0000 L CNN
-F 2 "" H 5650 5000 50  0001 C CNN
+F 2 "Capacitor_SMD:C_0603_1608Metric" H 5650 5000 50  0001 C CNN
 F 3 "~" H 5650 5000 50  0001 C CNN
 	1    5650 5000
@@
 F 0 "C1" H 1515 1346 50  0000 L CNN
 F 1 "10uF" H 1515 1255 50  0000 L CNN
-F 2 "" H 1400 1300 50  0001 C CNN
+F 2 "Capacitors_Tantalum_SMD:CP_Tantalum_Case-B_EIA-3528-21_Reflow" H 1400 1300 50  0001 C CNN
 F 3 "~" H 1400 1300 50  0001 C CNN
 	1    1400 1300
@@
 F 0 "C2" H 2515 1346 50  0000 L CNN
 F 1 "10uF" H 2515 1255 50  0000 L CNN
-F 2 "" H 2400 1300 50  0001 C CNN
+F 2 "Capacitors_Tantalum_SMD:CP_Tantalum_Case-B_EIA-3528-21_Reflow" H 2400 1300 50  0001 C CNN
 F 3 "~" H 2400 1300 50  0001 C CNN
 	1    2400 1300

Commit message: started working on keychain
Parts:
- removed U3: ATTINY13A-MU, QFN_MLF20, symbol MCU_Atmel_ATTINY:ATTINY13A-MU
- added U4: ATTINY13A-MMF, Package_DFN_QFN:DFN-10-1EP_3x3mm_P0.5mm_EP1.55x2.48mm, symbol atmel:ATTINY13A-MMF
- J1: footprint Pin_Headers:Pin_Header_Straight_2x03_Pitch2.54mm -> Connector_PinHeader_2.54mm:PinHeader_2x03_P2.54mm_Vertical
- SW1: footprint Buttons_Switches_SMD:SW_MEC_5GSH9 -> Button_Switch_SMD:SW_SPST_B3U-1000P
- U1: symbol Regulator_Linear:MIC5205-2.5 -> keychain_game-rescue:MIC5205-2.5-Regulator_Linear
- U2: footprint SOIC127P600X175-16N -> Package_SO:SOIC-16W_5.3x10.2mm_P1.27mm; symbol SN74HC595DR:SN74HC595DR -> keychain_game-rescue:SN74HC595DR-SN74HC595DR
Connections:
- net +2V5: now also U4.10 (VCC)
- net GND: now also U4.5 (GND)
- net MISO: now also U4.7 (PB1(MISO/AIN1/OC0B/INT0/PCINT1))
- net MOSI: now also U4.6 (PB0(MOSI/AIN0/OC0A/PCINT0))
- net RCLK: now also U4.9 (PB2(SCK/ADC1/T0/PCINT2))
- net RESET: now also U4.1 (PB5(~RESET~/ADC0/PCINT5/dW))
- net at R1.1, SW1.3 (B), SW1.4 (B): now also U4.4 (PB4(ADC2/PCINT4))
Changed lines of the file:
@@
 $EndDescr
-$Comp
-L MCU_Atmel_ATTINY:ATTINY13A-MU U3
-U 1 1 5B7E44F0
-P 4650 4400
-F 0 "U3" H 4650 4917 50  0000 C CNN
-F 1 "ATTINY13A-MU" H 4650 4826 50  0000 C CNN
-F 2 "QFN_MLF20" H 5300 4400 50  0001 C CIN
-F 3 "http://ww1.microchip.com/downloads/en/DeviceDoc/doc8126.pdf" H 3850 4750 50  0001 C CNN
-	1    4650 4400
-	1    0    0    -1
-$EndComp
 $Comp
 L power:+2V5 #PWR0101
@@
 $EndComp
 $Comp
-L SN74HC595DR:SN74HC595DR U2
+L keychain_game-rescue:SN74HC595DR-SN74HC595DR U2
 U 1 1 5B7E54FD
 P 4100 2250
 F 0 "U2" H 4100 3020 50  0000 C CNN
 F 1 "SN74HC595DR" H 4100 2929 50  0000 C CNN
-F 2 "SOIC127P600X175-16N" H 4100 2250 50  0001 L BNN
+F 2 "Package_SO:SOIC-16W_5.3x10.2mm_P1.27mm" H 4100 2250 50  0001 L BNN
 F 3 "Texas Instruments" H 4100 2250 50  0001 L BNN
 F 4 "SOIC-16 Texas Instruments" H 4100 2250 50  0001 L BNN "Field4"
@@
 F 0 "J1" H 4050 5417 50  0000 C CNN
 F 1 "Conn_02x03_Counter_Clockwise" H 4050 5326 50  0000 C CNN
-F 2 "Pin_Headers:Pin_Header_Straight_2x03_Pitch2.54mm" H 4000 5100 50  0001 C CNN
+F 2 "Connector_PinHeader_2.54mm:PinHeader_2x03_P2.54mm_Vertical" H 4000 5100 50  0001 C CNN
 F 3 "~" H 4000 5100 50  0001 C CNN
 	1    4000 5100
@@
 F 0 "SW1" V 2046 4702 50  0000 R CNN
 F 1 "SW_MEC_5G" V 1955 4702 50  0000 R CNN
-F 2 "Buttons_Switches_SMD:SW_MEC_5GSH9" H 2000 4950 50  0001 C CNN
+F 2 "Button_Switch_SMD:SW_SPST_B3U-1000P" H 2000 4950 50  0001 C CNN
 F 3 "http://www.apem.com/int/index.php?controller=attachment&id_attachment=488" H 2000 4950 50  0001 C CNN
 	1    2000 4750
@@
 RESET
 $Comp
-L Regulator_Linear:MIC5205-2.5 U1
+L keychain_game-rescue:MIC5205-2.5-Regulator_Linear U1
 U 1 1 5B7EA4B7
 P 1950 1250
@@
 	-1   0    0    1
 $EndComp
-Wire Wire Line
-	5650 4650 5650 4900
-Connection ~ 5650 4650
 $Comp
 L Device:CP1 C1
@@
 	0    -1   -1   0
 $EndComp
+Wire Wire Line
+	5650 4650 5650 4900
+Connection ~ 5650 4650
+$Comp
+L atmel:ATTINY13A-MMF U4
+U 1 1 5B8A0656
+P 4650 4400
+F 0 "U4" H 4650 4917 50  0000 C CNN
+F 1 "ATTINY13A-MMF" H 4650 4826 50  0000 C CNN
+F 2 "Package_DFN_QFN:DFN-10-1EP_3x3mm_P0.5mm_EP1.55x2.48mm" H 5250 4400 50  0001 C CIN
+F 3 "http://www.atmel.com/Images/doc8126.pdf" H 3850 4750 50  0001 C CNN
+	1    4650 4400
+	1    0    0    -1
+$EndComp
 $EndSCHEMATC

Commit message: finished board
Parts:
- removed SW1: SW_MEC_5G, Button_Switch_SMD:SW_SPST_B3U-1000P, symbol Switch:SW_MEC_5G
- added SW2: SW_DPST_x2, Button_Switch_SMD:SW_SPST_B3U-1000P, symbol Switch:SW_DPST_x2
Connections:
- net GND: now also SW2.2 (B)
- net MISO: now also U2.12 (RCLK); no longer U2.11 (SRCLK)
- net at R1.1, U4.4 (PB4(ADC2/PCINT4)): now also SW2.1 (A)
- net RCLK renamed SCK
- net SCK: now also U2.11 (SRCLK); no longer U2.12 (RCLK)
Changed lines of the file:
@@
 Text GLabel 3400 2050 0    50   Input ~ 0
 RCLK
+Text GLabel 1900 4250 0    50   Input ~ 0
+RCLK
 Text GLabel 1900 4350 0    50   Input ~ 0
-RCLK
-Text GLabel 1900 4250 0    50   Input ~ 0
 SRCLK
 Text GLabel 1900 4150 0    50   Input ~ 0
@@
 F 3 "" H 1600 4550 50  0001 C CNN
 	1    1600 4550
-	0    -1   -1   0
-$EndComp
-$Comp
-L Switch:SW_MEC_5G SW1
-U 1 1 5B7E7332
-P 2000 4750
-F 0 "SW1" V 2046 4702 50  0000 R CNN
-F 1 "SW_MEC_5G" V 1955 4702 50  0000 R CNN
-F 2 "Button_Switch_SMD:SW_SPST_B3U-1000P" H 2000 4950 50  0001 C CNN
-F 3 "http://www.apem.com/int/index.php?controller=attachment&id_attachment=488" H 2000 4950 50  0001 C CNN
-	1    2000 4750
 	0    -1   -1   0
 $EndComp
@@
 	1    0    0    -1
 $EndComp
+$Comp
+L Switch:SW_DPST_x2 SW2
+U 1 1 5B8A0B61
+P 2000 4750
+F 0 "SW2" V 1954 4848 50  0000 L CNN
+F 1 "SW_DPST_x2" V 2045 4848 50  0000 L CNN
+F 2 "Button_Switch_SMD:SW_SPST_B3U-1000P" H 2000 4750 50  0001 C CNN
+F 3 "" H 2000 4750 50  0001 C CNN
+	1    2000 4750
+	0    1    1    0
+$EndComp
 $EndSCHEMATC
